File: Esp32C6-Chinebasto.kicad_sch (KiCad schematic)
At the start: 3 parts, among them U1 ESP32-C6-WROOM-1-N8, U2 SN74LVC1G32DCKR, U4 SN74LVC2G32DCTR

Commit message: just started
Parts:
- added U3: AMS1117-3.3, Package_TO_SOT_SMD:SOT-223-3_TabPin2, symbol Regulator_Linear:AMS1117-3.3
- added U5: XD-XHD-2*2A, kicad-libraries:CONN-TH_XD-XHD-2-2A, symbol iu3qez:XD-XHD-2*2A
- added U6: CH340G, kicad-libraries:SOIC-16_L9.9-W3.9-P1.27-LS6.0-BL, symbol iu3qez:CH340G
- added USBC1: TYPE-C-31-M-12, kicad-libraries:USB-C_SMD-TYPE-C-31-M-12_1, symbol iu3qez:TYPE-C-31-M-12
Connections:
- new net +5V: U5.2
- new net Blu: U5.3
- new net GND: U3.1 (GND), U5.1
- no-connect marks 0 -> 1
Other:
- moved on the sheet: U4

Commit message: updatee
Parts:
- removed U3: AMS1117-3.3, Package_TO_SOT_SMD:SOT-223-3_TabPin2, symbol Regulator_Linear:AMS1117-3.3
- added C1, C2: 2.2uF, Capacitor_SMD:C_0805_2012Metric_Pad1.18x1.45mm_HandSolder, symbol Device:C
- added U1: SGM2212-3.3XKC3G/TR_C3294699, kicad-libraries:SOT-223-3_L6.5-W3.4-P2.30-LS7.0-BR, symbol LIbreire IU3qez:SGM2212-3.3XKC3G_TR_C3294699
Connections:
- net +5V: now also U2.5 (VCC)
- net GND: now also U6.1 (GND), C1.2, C2.2, U1.1 (GND)
- new net 3.3V: C2.1, U1.2 (VOUT), U1.4 (VOUT)
- new net VCC: C1.1, U1.3 (VIN)
Other:
- moved on the sheet: U1

Commit message: Update
Parts:
- renumbered U4 to U1, U1 to U3, U5 to U4, U1 to U5
Changed lines of the file:
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@@
 		(in_pos_files yes)
 		(dnp no)
-		(property "Reference" "#PWR01"
+		(property "Reference" "#PWR05"
 			(at 144.78 127 0)
 			(hide yes)
@@
 			(project ""
 				(path "/75db8882-5d53-4ed0-a3d0-0bb6372cd542"
-					(reference "#PWR01")
+					(reference "#PWR05")
 					(unit 1)
 				)
@@
 		(dnp no)
 		(fields_autoplaced yes)
-		(property "Reference" "#PWR01"
+		(property "Reference" "#PWR02"
 			(at 135.89 55.88 0)
 			(hide yes)
@@
 			(project ""
 				(path "/75db8882-5d53-4ed0-a3d0-0bb6372cd542"
-					(reference "#PWR01")
+					(reference "#PWR02")
 					(unit 1)
 				)
@@
 		(dnp no)
 		(fields_autoplaced yes)
-		(property "Reference" "#PWR03"
+		(property "Reference" "#PWR04"
 			(at 147.32 50.8 0)
 			(hide yes)
@@
 			(project ""
 				(path "/75db8882-5d53-4ed0-a3d0-0bb6372cd542"
-					(reference "#PWR03")
+					(reference "#PWR04")
 					(unit 1)
 				)
@@
 		(dnp no)
 		(fields_autoplaced yes)
-		(property "Reference" "#PWR02"
+		(property "Reference" "#PWR03"
 			(at 142.24 48.26 0)
 			(hide yes)
@@
 			(project ""
 				(path "/75db8882-5d53-4ed0-a3d0-0bb6372cd542"
-					(reference "#PWR02")
+					(reference "#PWR03")
 					(unit 1)
 				)
@@
 		(dnp no)
 		(fields_autoplaced yes)
-		(property "Reference" "#PWR05"
+		(property "Reference" "#PWR08"
 			(at 186.69 46.99 0)
 			(hide yes)
@@
 			(project ""
 				(path "/75db8882-5d53-4ed0-a3d0-0bb6372cd542"
-					(reference "#PWR05")
+					(reference "#PWR08")
 					(unit 1)
 				)
@@
 		(dnp no)
 		(fields_autoplaced yes)
-		(property "Reference" "#PWR02"
+		(property "Reference" "#PWR06"
 			(at 151.13 125.73 0)
 			(hide yes)
@@
 			(project ""
 				(path "/75db8882-5d53-4ed0-a3d0-0bb6372cd542"
-					(reference "#PWR02")
+					(reference "#PWR06")
 					(unit 1)
 				)
@@
 		(dnp no)
 		(fields_autoplaced yes)
-		(property "Reference" "U1"
+		(property "Reference" "U5"
 			(at 162.56 36.83 0)
 			(show_name no)
@@
 			(project ""
 				(path "/75db8882-5d53-4ed0-a3d0-0bb6372cd542"
-					(reference "U1")
+					(reference "U5")
 					(unit 1)
 				)
@@
 		(dnp no)
 		(fields_autoplaced yes)
-		(property "Reference" "U1"
+		(property "Reference" "U3"
 			(at 92.71 81.28 0)
 			(show_name no)
@@
 			(project ""
 				(path "/75db8882-5d53-4ed0-a3d0-0bb6372cd542"
-					(reference "U1")
+					(reference "U3")
 					(unit 1)
 				)
@@
 		(dnp no)
 		(fields_autoplaced yes)
-		(property "Reference" "#PWR010"
+		(property "Reference" "#PWR01"
 			(at 104.14 113.03 0)
 			(hide yes)
@@
 			(project "Esp32C6-Chinebasto"
 				(path "/75db8882-5d53-4ed0-a3d0-0bb6372cd542"
-					(reference "#PWR010")
+					(reference "#PWR01")
 					(unit 1)
 				)
@@
 		(dnp no)
 		(fields_autoplaced yes)
-		(property "Reference" "U4"
+		(property "Reference" "U1"
 			(at 55.88 105.41 0)
 			(show_name no)
@@
 			(project ""
 				(path "/75db8882-5d53-4ed0-a3d0-0bb6372cd542"
-					(reference "U4")
+					(reference "U1")
 					(unit 1)
 				)
@@
 		(dnp no)
 		(fields_autoplaced yes)
-		(property "Reference" "U5"
+		(property "Reference" "U4"
 			(at 156.21 119.38 0)
 			(show_name no)
@@
 			(project ""
 				(path "/75db8882-5d53-4ed0-a3d0-0bb6372cd542"
-					(reference "U5")
+					(reference "U4")
 					(unit 1)
 				)
@@
 		(dnp no)
 		(fields_autoplaced yes)
-		(property "Reference" "#PWR04"
+		(property "Reference" "#PWR07"
 			(at 176.53 48.26 0)
 			(hide yes)
@@
 			(project ""
 				(path "/75db8882-5d53-4ed0-a3d0-0bb6372cd542"
-					(reference "#PWR04")
+					(reference "#PWR07")
 					(unit 1)
 				)
@@
 		(dnp no)
 		(fields_autoplaced yes)
-		(property "Reference" "#PWR09"
+		(property "Reference" "#PWR012"
 			(at 213.36 63.5 0)
 			(hide yes)
@@
 			(project ""
 				(path "/75db8882-5d53-4ed0-a3d0-0bb6372cd542"
-					(reference "#PWR09")
+					(reference "#PWR012")
 					(unit 1)
 				)
@@
 		(dnp no)
 		(fields_autoplaced yes)
-		(property "Reference" "#PWR07"
+		(property "Reference" "#PWR010"
 			(at 203.2 46.99 0)
 			(hide yes)
@@
 			(project ""
 				(path "/75db8882-5d53-4ed0-a3d0-0bb6372cd542"
-					(reference "#PWR07")
+					(reference "#PWR010")
 					(unit 1)
 				)
@@
 		(dnp no)
 		(fields_autoplaced yes)
-		(property "Reference" "#PWR08"
+		(property "Reference" "#PWR011"
 			(at 203.2 57.15 0)
 			(hide yes)
@@
 			(project ""
 				(path "/75db8882-5d53-4ed0-a3d0-0bb6372cd542"
-					(reference "#PWR08")
+					(reference "#PWR011")
 					(unit 1)
 				)
@@
 		(dnp no)
 		(fields_autoplaced yes)
-		(property "Reference" "#PWR06"
+		(property "Reference" "#PWR09"
 			(at 186.69 57.15 0)
 			(hide yes)
@@
 			(project ""
 				(path "/75db8882-5d53-4ed0-a3d0-0bb6372cd542"
-					(reference "#PWR06")
-					(unit 1)
-				)
+					(reference "#PWR09")
+					(unit 1)
+				)

Commit message: Update
Parts:
- added D1, D2, D3: 1N4148W, Diode_SMD:D_SOD-123, symbol Diode:1N4148W
- added USBC2: TYPE-C-31-M-12, kicad-libraries:USB-C_SMD-TYPE-C-31-M-12_1, symbol iu3qez:TYPE-C-31-M-12
- added X1: X322512MSB4SI, kicad-libraries:CRYSTAL-SMD_4P-L3.2-W2.5-BL, symbol iu3qez:X322512MSB4SI
Connections:
- net +5V: now also D1.2 (A)
- net GND: now also USBC1.1 (EH), USBC1.2 (EH), USBC1.3 (EH), USBC1.4 (EH), USBC1.A1B12 (GND), USBC1.B1A12 (GND), USBC2.1 (EH), USBC2.2 (EH), USBC2.3 (EH), USBC2.4 (EH), USBC2.A1B12 (GND), USBC2.B1A12 (GND), X1.2 (GND), X1.4 (GND)
- net Vcc: now reaches U6.16 (VCC)
- net Vcc: now also D1.1 (K), D2.1 (K), D3.1 (K)
- net TX: now reaches U6.2 (TXD)
- net RX: now reaches U6.3 (RXD)
- net at U6.7 (XI): now also X1.3 (OSC2)
- net at U6.8 (XO): now also X1.1 (OSC1)
- net USB2_N: now reaches U3.13 (IO12)
- net USB2_P: now reaches U3.14 (IO13)
- net VBUS1: now reaches USBC1.A4B9 (VBUS)
- net VBUS1: now also USBC1.B4A9 (VBUS), D3.2 (A)
- net USB1_P: now reaches USBC1.A6 (DP1)
- net USB1_P: now also USBC1.B6 (DP2)
- net USB1_N: now reaches USBC1.A7 (DN1)
- net USB1_N: now also USBC1.B7 (DN2)
- new net VBUS2: D2.2 (A)
Other:
- moved on the sheet: USBC1

Commit message: update
Parts:
- removed D1, D2, D3: 1N4148W, Diode_SMD:D_SOD-123, symbol Diode:1N4148W
- removed U6: CH340G, kicad-libraries:SOIC-16_L9.9-W3.9-P1.27-LS6.0-BL, symbol iu3qez:CH340G
- removed USBC1: TYPE-C-31-M-12, kicad-libraries:USB-C_SMD-TYPE-C-31-M-12_1, symbol iu3qez:TYPE-C-31-M-12
- removed X1: X322512MSB4SI, kicad-libraries:CRYSTAL-SMD_4P-L3.2-W2.5-BL, symbol iu3qez:X322512MSB4SI
- added C3: C_Small, Capacitor_SMD:C_0603_1608Metric_Pad1.08x0.95mm_HandSolder, symbol Device:C_Small
- added C4, C5: 10p, Capacitor_SMD:C_0603_1608Metric_Pad1.08x0.95mm_HandSolder, symbol Device:C_Small
- added D1, D2, D3: D_Schottky, symbol Device:D_Schottky
- added R1, R2: 5.1k, Resistor_SMD:R_0603_1608Metric_Pad0.98x0.95mm_HandSolder, symbol Device:R_Small
- added U6: CH340G, Z_IU3qez:SOIC-16_L9.9-W3.9-P1.27-LS6.0-BL, symbol Interface_USB:CH340G
- added USBC2: C165948, Z_IU3qez:USB-C_SMD-TYPE-C-31-M-12_1, symbol USB:TYPE-C-31-M-12
- added Y1: 12MHz, Z_IU3qez:CRYSTAL-SMD_4P-L3.2-W2.5-BL, symbol PCM_SparkFun-Clock:Crystal_12MHz_2.5x2.0mm
- U1: footprint kicad-libraries:SM-8_L3.0-W2.8-P0.65-LS4.0-BL -> Z_IU3qez:SM-8_L3.0-W2.8-P0.65-LS4.0-BL
- U2: footprint kicad-libraries:SC-70-5_L2.0-W1.3-P0.65-LS2.1-BR -> Z_IU3qez:SC-70-5_L2.0-W1.3-P0.65-LS2.1-BR
- U3: footprint kicad-libraries:WIRELM-SMD_ESP32-C6-WROOM-1 -> Z_IU3qez:WIRELM-SMD_ESP32-C6-WROOM-1
- U4: footprint kicad-libraries:CONN-TH_XD-XHD-2-2A -> Z_IU3qez:CONN-TH_XD-XHD-2-2A
- U5: footprint kicad-libraries:SOT-223-3_L6.5-W3.4-P2.30-LS7.0-BR -> Z_IU3qez:SOT-223-3_L6.5-W3.4-P2.30-LS7.0-BR
- USBC1: renamed from USBC2; footprint kicad-libraries:USB-C_SMD-TYPE-C-31-M-12_1 -> Z_IU3qez:USB-C_SMD-TYPE-C-31-M-12_1
Connections:
- net USB2_N is gone; now on net USB2-: U3.13 (IO12)
- net USB2_P is gone; now on net USB2+: U3.14 (IO13)
- net +5V: now also D1.2 (A); no longer U2.5 (VCC)
- net 3.3V: now also C3.1, U6.16 (VCC), U6.4 (V3)
- net GND: now also C3.2, C4.1, C5.2, R1.2, R2.2, U6.1 (GND), USBC2.1 (EH), USBC2.2 (EH), USBC2.3 (EH), USBC2.4 (EH), USBC2.A1B12 (GND), USBC2.B1A12 (GND), Y1.2, Y1.4
- net VBUS1: now also D3.2 (A), USBC2.A4B9 (VBUS), USBC2.B4A9 (VBUS)
- net VBUS2: now also USBC1.A4B9 (VBUS), USBC1.B4A9 (VBUS), D2.2 (A)
- net Vcc: now also U2.5 (VCC), D1.1 (K), D2.1 (K), D3.1 (K)
- net USB2+: now reaches USBC1.A6 (DP1)
- net USB2+: now also USBC1.B6 (DP2)
- net USB2-: now reaches USBC1.A7 (DN1)
- net USB2-: now also USBC1.B7 (DN2)
- new net: C5.1, U6.8 (XO), Y1.1
- new net: C4.2, U6.7 (XI), Y1.3
- new net: R2.1, USBC2.B5 (CC2)
- new net: R1.1, USBC2.A5 (CC1)
- new net D+: U6.5 (UD+), USBC2.A6 (DP1), USBC2.B6 (DP2)
- new net D-: U6.6 (UD-), USBC2.A7 (DN1), USBC2.B7 (DN2)
- new net DTR: U6.13 (~{DTR})
- new net ESP32_RX: U6.2 (TXD)
- new net ESP32_TX: U6.3 (RXD)
- new net RTS: U6.14 (~{RTS})
- no-connect marks 1 -> 8

Commit message: Update
Parts:
- removed U2: SN74LVC1G32DCKR, Z_IU3qez:SC-70-5_L2.0-W1.3-P0.65-LS2.1-BR, symbol iu3qez:SN74LVC1G32DCKR
- added C6, C7: 100n, Capacitor_SMD:C_0603_1608Metric_Pad1.08x0.95mm_HandSolder, symbol Device:C_Small
- added D4: D_Zener, Diode_SMD:D_MiniMELF_Handsoldering, symbol Device:D_Zener
- added R3: 470, Resistor_SMD:R_0603_1608Metric_Pad0.98x0.95mm_HandSolder, symbol Device:R_Small
- added U2: 74LVC1G126GW, Z_IU3qez:SOT-353-5_L2.0-W1.6-P0.65-LS2.1-BL, symbol iu3qez:74LVC1G126GW
- D1, D2, D3: footprint (none) -> Diode_SMD:D_SOD-123
Connections:
- net Blu: now also R3.2
- net GND: now also U1.4 (GND), U1.5 (2A), U1.6 (2B), C6.1, C7.1, D4.2 (A), U2.3 (GND)
- net Vcc: now also C7.2, U2.5 (VCC)
- net Chinebasto RX: now reaches U3.17 (IO19)
- net Chinebasto RX: now also U1.7 (1Y)
- net TxEn: now reaches U3.18 (IO20)
- net TxEn: now also U1.1 (1A), U2.1 (OE)
- net Chinebasto TX: now reaches U3.19 (IO21)
- net Chinebasto TX: now also U2.2 (A)
- net at U1.2 (1B): now also D4.1 (K), R3.1, U2.4 (Y)
- net +3.3V: now reaches U1.8 (VCC)
- net +3.3V: now also C6.2
- no-connect marks 8 -> 9

Commit message: update
Parts:
- added C8: 100n, Capacitor_SMD:C_0603_1608Metric_Pad1.08x0.95mm_HandSolder, symbol Device:C_Small
- added R4, R5: 470, Resistor_SMD:R_0603_1608Metric_Pad0.98x0.95mm_HandSolder, symbol Device:R_Small
- D4: footprint Diode_SMD:D_MiniMELF_Handsoldering -> Diode_SMD:D_MiniMELF
Connections:
- net +3.3V: now also U3.2 (3V3), C8.2
- net GND: now also C8.1, R4.1, R5.1
- net at USBC1.A5 (CC1): now also R5.2
- net at USBC1.B5 (CC2): now also R4.2
Other:
- moved on the sheet: C3, C4, C5, R1, R2, U6, USBC2, Y1

Commit message: update
Parts:
- added H1, H2, H3, H4: MountingHole_Pad, MountingHole:MountingHole_3.2mm_M3_ISO7380_Pad_TopBottom, symbol Mechanical:MountingHole_Pad
Connections:
- net 3.3V is gone; now on net +3.3V: C2.1, C3.1, U5.2 (VOUT), U5.4 (VOUT), U6.16 (VCC), U6.4 (V3)
- net GND: now also H1.1, H2.1, H3.1, H4.1
