File: Esp32C6-Chinebasto.kicad_sch (KiCad schematic)
At the start: 30 parts, among them U1 SN74LVC2G32DCTR, U2 74LVC1G126GW, U3 ESP32-C6-WROOM-1-N8, U4 XD-XHD-2*2A, U5 SGM2212-3.3XKC3G/TR_C3294699, U6 CH340G, Y1 12MHz

Commit message: update
Parts:
- added C9: 100n, Capacitor_SMD:C_0603_1608Metric_Pad1.08x0.95mm_HandSolder, symbol Device:C_Small
- added D5: LED, LED_SMD:LED_0603_1608Metric_Pad1.05x0.95mm_HandSolder, symbol Device:LED
- added Q1, Q2: MMBT3904, Package_TO_SOT_SMD:SOT-23, symbol Transistor_BJT:MMBT3904
- added R10, R11: 10k, Resistor_SMD:R_0603_1608Metric_Pad0.98x0.95mm_HandSolder, symbol Device:R_Small
- added R6, R7: 10k, Resistor_SMD:R_0603_1608Metric_Pad0.98x0.95mm_HandSolder, symbol Device:R
- added R8, R9: 0, Resistor_SMD:R_0603_1608Metric_Pad0.98x0.95mm_HandSolder, symbol Device:R
- added SW1, SW2, SW3: SW_Push, Switch_Keyboard_Kailh:SW_Kailh_Choc_V1V2_1.00u, symbol Switch:SW_Push
- renumbered C6 to C1, C7 to C2, C8 to C3, C1 to C4, C2 to C5, C3 to C6, C4 to C7, C5 to C8, D4 to D1, D1 to D2, D2 to D3, D3 to D4, H3 to H1, H4 to H2, H1 to H3, H2 to H4, R3 to R1, R5 to R2, R4 to R3, R1 to R4, R2 to R5
Connections:
- net +3.3V: now also R10.1
- net DTR: now also Q2.2 (E), R6.1
- net ESP32_RX: now also U3.25 (TXD0)
- net ESP32_TX: now also U3.24 (RXD0)
- net GND: now also U3.1 (GND), U3.28 (GND), U3.29 (GND), U3.30 (GND), U3.31 (GND), U3.32 (GND), U3.33 (GND), U3.34 (GND), U3.35 (GND), U3.36 (GND), U3.37 (GND), C9.1, D5.1 (K), SW1.2, SW2.2, SW3.2
- net RTS: now also Q1.2 (E), R7.1
- net at U3.11 (IO10): now also R11.1
- net at U3.20 (IO22): now also SW3.1
- net at U3.21 (IO23): now also SW2.1
- net at U3.23 (IO15): now also SW1.1
- net ESP32_EN: now reaches U3.3 (EN)
- net ESP32_EN: now also C9.2, R10.2, R8.2
- net ESP32_GPIO0: now reaches U3.8 (IO0)
- net ESP32_GPIO0: now also R9.2
- new net: D5.2 (A), R11.2
- new net: Q2.1 (B), R7.2
- new net: Q2.3 (C), R9.1
- new net: Q1.1 (B), R6.2
- new net: Q1.3 (C), R8.1
- no-connect marks 9 -> 10
