File: Esp32C6-Chinebasto.kicad_pcb (KiCad board)
At the start: 2 copper layers, 9 parts, among them U1 SN74LVC2G32DCTR, U2 SN74LVC1G32DCKR, U3 ESP32-C6-WROOM-1-N8, U4 XD-XHD-2*2A, U5 SGM2212-3.3XKC3G/TR_C3294699, U6 CH340G

Commit message: update
Parts:
- added C3: C_Small, Capacitor_SMD:C_0603_1608Metric_Pad1.08x0.95mm_HandSolder, F.Cu at (88.5, 122.3)
- added C4: 10p, Capacitor_SMD:C_0603_1608Metric_Pad1.08x0.95mm_HandSolder, F.Cu at (88.5, 124.8)
- added C5: 10p, Capacitor_SMD:C_0603_1608Metric_Pad1.08x0.95mm_HandSolder, F.Cu at (88.5, 127.3)
- added R1: 5.1k, Resistor_SMD:R_0603_1608Metric_Pad0.98x0.95mm_HandSolder, F.Cu at (88.5, 129.8)
- added R2: 5.1k, Resistor_SMD:R_0603_1608Metric_Pad0.98x0.95mm_HandSolder, F.Cu at (88.5, 132.3)
- added U6: CH340G, Z_IU3qez:SOIC-16_L9.9-W3.9-P1.27-LS6.0-BL, F.Cu at (92.4, 137.8)
- added USBC1: TYPE-C-31-M-12, Z_IU3qez:USB-C_SMD-TYPE-C-31-M-12_1, F.Cu at (80.9, 124.7)
- added USBC2: C165948, Z_IU3qez:USB-C_SMD-TYPE-C-31-M-12_1, F.Cu at (111.4, 126.7)
- added Y1: 12MHz, Z_IU3qez:CRYSTAL-SMD_4P-L3.2-W2.5-BL, F.Cu at (93.5, 123.3)
- U1: footprint kicad-libraries:SM-8_L3.0-W2.8-P0.65-LS4.0-BL -> Z_IU3qez:SM-8_L3.0-W2.8-P0.65-LS4.0-BL
- U2: footprint kicad-libraries:SC-70-5_L2.0-W1.3-P0.65-LS2.1-BR -> Z_IU3qez:SC-70-5_L2.0-W1.3-P0.65-LS2.1-BR
- U3: footprint kicad-libraries:WIRELM-SMD_ESP32-C6-WROOM-1 -> Z_IU3qez:WIRELM-SMD_ESP32-C6-WROOM-1
- U4: footprint kicad-libraries:CONN-TH_XD-XHD-2-2A -> Z_IU3qez:CONN-TH_XD-XHD-2-2A
- U5: footprint kicad-libraries:SOT-223-3_L6.5-W3.4-P2.30-LS7.0-BR -> Z_IU3qez:SOT-223-3_L6.5-W3.4-P2.30-LS7.0-BR
- moved U1 15.6 mm to (101.5, 124.6)
Connections:
- U2 pad 5: +5V -> /Vcc
- U3 pad 13: unconnected-(U3-IO12-Pad13) -> /USB2-
- U3 pad 14: unconnected-(U3-IO13-Pad14) -> /USB2+

Commit message: Update
Parts:
- removed the USBC1 at (116.4, 83.2)
- added C6: 100n, Capacitor_SMD:C_0603_1608Metric_Pad1.08x0.95mm_HandSolder, F.Cu at (126.0, 144.6)
- added C7: 100n, Capacitor_SMD:C_0603_1608Metric_Pad1.08x0.95mm_HandSolder, F.Cu at (126.0, 147.1)
- added D1: D_Schottky, Diode_SMD:D_SOD-123, F.Cu at (120.9, 145.0)
- added D2: D_Schottky, Diode_SMD:D_SOD-123, F.Cu at (120.9, 148.4)
- added D3: D_Schottky, Diode_SMD:D_SOD-123, F.Cu at (120.9, 151.7)
- added D4: D_Zener, Diode_SMD:D_MiniMELF_Handsoldering, F.Cu at (123.2, 141.7)
- added R3: 470, Resistor_SMD:R_0603_1608Metric_Pad0.98x0.95mm_HandSolder, F.Cu at (126.0, 149.6)
- U2: value SN74LVC1G32DCKR -> 74LVC1G126GW; footprint Z_IU3qez:SC-70-5_L2.0-W1.3-P0.65-LS2.1-BR -> Z_IU3qez:SOT-353-5_L2.0-W1.6-P0.65-LS2.1-BL
- moved USBC2 44.8 mm to (81.5, 160.0)
- turned USBC1 to -90 degrees
Connections:
- U1 pad 1: unconnected-(U1-1A-Pad1) -> /TxEn
- U1 pad 2: unconnected-(U1-1B-Pad2) -> Net-(D4-K)
- U1 pad 4: unconnected-(U1-GND-Pad4) -> GND
- U1 pad 5: unconnected-(U1-2A-Pad5) -> GND
- U1 pad 6: unconnected-(U1-2B-Pad6) -> GND
- U1 pad 7: unconnected-(U1-1Y-Pad7) -> /Chinebasto RX
- U1 pad 8: unconnected-(U1-VCC-Pad8) -> +3.3V
- U2 pad 1: unconnected-(U2-A-Pad1) -> /TxEn
- U2 pad 2: unconnected-(U2-B-Pad2) -> /Chinebasto TX
- U2 pad 3: unconnected-(U2-GND-Pad3) -> GND
- U2 pad 4: unconnected-(U2-Y-Pad4) -> Net-(D4-K)
- U3 pad 17: unconnected-(U3-IO19-Pad17) -> /Chinebasto RX
- U3 pad 18: unconnected-(U3-IO20-Pad18) -> /TxEn
- U3 pad 19: unconnected-(U3-IO21-Pad19) -> /Chinebasto TX
Other:
- board outline added: 60 x 60 mm

Commit message: update
Parts:
- removed the U6 at (136.0, 100.2)
- added R4: 470, Resistor_SMD:R_0603_1608Metric_Pad0.98x0.95mm_HandSolder, F.Cu at (78.4, 141.0)
- added R5: 470, Resistor_SMD:R_0603_1608Metric_Pad0.98x0.95mm_HandSolder, F.Cu at (58.3, 142.2)
- D4: footprint Diode_SMD:D_MiniMELF_Handsoldering -> Diode_SMD:D_MiniMELF
- moved C2 78.0 mm to (53.0, 125.5), turned to 90 degrees
- moved U5 71.5 mm to (59.5, 125.5), turned to -90 degrees
- moved C1 66.1 mm to (65.5, 125.5), turned to 90 degrees
- moved R3 58.5 mm to (96.9, 98.8)
- moved C7 54.1 mm to (97.7, 101.0)
- moved C6 49.4 mm to (93.7, 107.2)
- moved D2 46.1 mm to (77.2, 133.7), turned to -90 degrees
- moved D3 44.2 mm to (80.6, 133.7), turned to -90 degrees
- moved D4 39.1 mm to (102.4, 108.6), turned to -90 degrees
- moved D1 39.0 mm to (107.6, 108.4), turned to 90 degrees
- moved USBC1 23.8 mm to (68.5, 145.0), turned to 0 degrees
- moved U3 22.5 mm to (80.8, 105.8)
- moved U1 21.4 mm to (96.5, 103.8), turned to 90 degrees
- moved USBC2 18.3 mm to (92.0, 145.0)
- moved U4 12.6 mm to (103.3, 97.5)
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Connections:
- USBC1 pad A5: unconnected-(USBC1-CC1-PadA5) -> Net-(USBC1-CC1)
- USBC1 pad B5: unconnected-(USBC1-CC2-PadB5) -> Net-(USBC1-CC2)
Routing:
- net /USB2-: track 0.00 -> 33.3 mm
- net /USB2+: track 0.00 -> 32.5 mm
- net /VBUS2: track 0.00 -> 22.3 mm, vias 0 -> 2
- net Net-(D4-K): track 0.00 -> 19.9 mm
- net /VBUS1: track 0.00 -> 19.6 mm
- net /D-: track 0.00 -> 18.3 mm
- net 3.3V: track 0.00 -> 18.2 mm
- net /TxEn: track 0.00 -> 17.3 mm, vias 0 -> 2
- net /Chinebasto RX: track 0.00 -> 15.7 mm
- net /D+: track 0.00 -> 15.1 mm
- net /Vcc: track 0.00 -> 14.4 mm, vias 0 -> 2
- net Net-(USBC1-CC1): track 0.00 -> 13.3 mm
- net Net-(USBC1-CC2): track 0.00 -> 11.7 mm
- net +5V: track 0.00 -> 11.7 mm
- net /Chinebasto TX: track 0.00 -> 6.57 mm
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Other:
- outline, holes or cut-outs redrawn
- board text added: "Main Sheet"

Commit message: update
Parts:
- added C8: 100n, Capacitor_SMD:C_0603_1608Metric_Pad1.08x0.95mm_HandSolder, F.Cu at (67.0, 99.9)
- added H1: MountingHole_Pad, MountingHole:MountingHole_3.2mm_M3_ISO7380_Pad_TopBottom, F.Cu at (53.5, 93.5)
- added H2: MountingHole_Pad, MountingHole:MountingHole_3.2mm_M3_ISO7380_Pad_TopBottom, F.Cu at (53.5, 146.6)
- added H3: MountingHole_Pad, MountingHole:MountingHole_3.2mm_M3_ISO7380_Pad_TopBottom, F.Cu at (106.5, 93.5)
- added H4: MountingHole_Pad, MountingHole:MountingHole_3.2mm_M3_ISO7380_Pad_TopBottom, F.Cu at (106.5, 146.6)
- moved C4 10.1 mm to (98.4, 122.5), turned to 180 degrees
- moved R3 7.01 mm to (103.6, 100.9), turned to 90 degrees
- moved U4 6.14 mm to (97.5, 95.8), turned to 180 degrees
- moved C7 6.10 mm to (100.0, 106.6), turned to -90 degrees
- moved C5 4.25 mm to (89.5, 123.1), turned to 90 degrees
Connections:
- C2 pad 1: 3.3V -> +3.3V
- C3 pad 1: 3.3V -> +3.3V
- U3 pad 2: unconnected-(U3-3V3-Pad2) -> +3.3V
- U5 pad 2: 3.3V -> +3.3V
- U5 pad 4: 3.3V -> +3.3V
- U6 pad 16: 3.3V -> +3.3V
- U6 pad 4: 3.3V -> +3.3V
Routing:
- net +3.3V: track 2.44 -> 125.1 mm, vias 0 -> 4
- net /Vcc: track 14.4 -> 47.6 mm
- net 3.3V: track 18.2 -> 0.00 mm
- net (no net): track 0.00 -> 12.4 mm
- net Net-(U6-XI): track 0.00 -> 8.91 mm
- net Net-(U6-XO): track 0.00 -> 7.29 mm
- net Net-(USBC2-CC2): track 0.00 -> 7.03 mm
- net /VBUS2: track 22.3 -> 16.9 mm
- net +5V: track 11.7 -> 15.4 mm
- net /Blu: track 4.27 -> 7.43 mm
- net Net-(D4-K): track 19.9 -> 18.0 mm, vias 0 -> 2
- net /D+: track 15.1 -> 16.7 mm
- net /USB2-: track 33.3 -> 34.2 mm
- net /D-: track 18.3 -> 19.0 mm
- net GND: vias 0 -> 9
- added copper zone on B.Cu, net GND
- added copper zone on F.Cu, net GND

Commit message: update
Parts:
- added C9: 100n, Capacitor_SMD:C_0603_1608Metric_Pad1.08x0.95mm_HandSolder, F.Cu at (69.4, 102.5)
- added D5: LED, LED_SMD:LED_0603_1608Metric_Pad1.05x0.95mm_HandSolder, F.Cu at (63.4, 113.7)
- added Q1: MMBT3904, Package_TO_SOT_SMD:SOT-23, F.Cu at (85.5, 126.4)
- added Q2: MMBT3904, Package_TO_SOT_SMD:SOT-23, F.Cu at (76.0, 126.6)
- added R10: 10k, Resistor_SMD:R_0603_1608Metric_Pad0.98x0.95mm_HandSolder, F.Cu at (67.0, 104.9)
- added R11: 10k, Resistor_SMD:R_0603_1608Metric_Pad0.98x0.95mm_HandSolder, F.Cu at (63.4, 109.9)
- added R6: 10k, Resistor_SMD:R_0603_1608Metric_Pad0.98x0.95mm_HandSolder, F.Cu at (82.6, 129.2)
- added R7: 10k, Resistor_SMD:R_0603_1608Metric_Pad0.98x0.95mm_HandSolder, F.Cu at (72.0, 129.4)
- added R8: 0, Resistor_SMD:R_0603_1608Metric_Pad0.98x0.95mm_HandSolder, F.Cu at (83.0, 121.9)
- added R9: 0, Resistor_SMD:R_0603_1608Metric_Pad0.98x0.95mm_HandSolder, F.Cu at (76.0, 121.9)
- added SW1: SW_Push, Switch_Keyboard_Kailh:SW_Kailh_Choc_V1V2_1.00u, F.Cu at (111.5, 103.4)
- added SW2: SW_Push, Switch_Keyboard_Kailh:SW_Kailh_Choc_V1V2_1.00u, F.Cu at (111.5, 120.8)
- added SW3: SW_Push, Switch_Keyboard_Kailh:SW_Kailh_Choc_V1V2_1.00u, F.Cu at (111.5, 138.0)
- moved D2 16.6 mm to (104.8, 92.0), turned to 180 degrees
- moved H2 16.1 mm to (122.6, 146.4)
- moved H1 15.9 mm to (122.4, 93.4)
- moved R1 14.5 mm to (92.0, 92.3)
- moved D1 6.17 mm to (99.8, 114.2)
- renumbered C6 to C1, C7 to C2, C8 to C3, C1 to C4, C2 to C5, C3 to C6, C4 to C7, C5 to C8, D4 to D1, D1 to D2, D2 to D3, D3 to D4, H3 to H1, H4 to H2, H1 to H3, H2 to H4, R3 to R1, R5 to R2, R4 to R3, R1 to R4, R2 to R5
Connections:
- U3 pad 1: unconnected-(U3-GND-Pad1) -> GND
- U3 pad 11: unconnected-(U3-IO10-Pad11) -> Net-(U3-IO10)
- U3 pad 20: unconnected-(U3-IO22-Pad20) -> Net-(U3-IO22)
- U3 pad 21: unconnected-(U3-IO23-Pad21) -> Net-(U3-IO23)
- U3 pad 23: unconnected-(U3-IO15-Pad23) -> Net-(U3-IO15)
- U3 pad 24: unconnected-(U3-RXD0-Pad24) -> ESP32_TX
- U3 pad 25: unconnected-(U3-TXD0-Pad25) -> ESP32_RX
- U3 pad 28: unconnected-(U3-GND-Pad28) -> GND
- U3 pad 29: unconnected-(U3-GND-Pad29) -> GND
- U3 pad 3: unconnected-(U3-EN-Pad3) -> ESP32_EN
- U3 pad 30: unconnected-(U3-GND-Pad30) -> GND
- U3 pad 31: unconnected-(U3-GND-Pad31) -> GND
- U3 pad 32: unconnected-(U3-GND-Pad32) -> GND
- U3 pad 33: unconnected-(U3-GND-Pad33) -> GND
- U3 pad 34: unconnected-(U3-GND-Pad34) -> GND
- U3 pad 35: unconnected-(U3-GND-Pad35) -> GND
- U3 pad 36: unconnected-(U3-GND-Pad36) -> GND
- U3 pad 37: unconnected-(U3-GND-Pad37) -> GND
- U3 pad 8: unconnected-(U3-IO0-Pad8) -> ESP32_GPIO0
Routing:
- net ESP32_RX: track 0.00 -> 45.1 mm, vias 0 -> 2
- net Net-(U3-IO22): track 0.00 -> 44.7 mm, vias 0 -> 2
- net GND: track 2.89 -> 46.4 mm, vias 9 -> 24
- net ESP32_TX: track 0.00 -> 39.2 mm, vias 0 -> 2
- net ESP32_EN: track 0.00 -> 38.4 mm, vias 0 -> 2
- net Net-(U3-IO23): track 0.00 -> 37.6 mm, vias 0 -> 2
- net Net-(U3-IO15): track 0.00 -> 26.6 mm, vias 0 -> 2
- net RTS: track 0.00 -> 22.2 mm, vias 0 -> 2
- net ESP32_GPIO0: track 0.00 -> 16.8 mm
- net DTR: track 0.00 -> 16.3 mm, vias 0 -> 3
- net /Vcc: track 47.6 -> 59.3 mm
- net +3.3V: track 125.1 -> 135.0 mm
- net Net-(U3-IO10): track 0.00 -> 9.11 mm, vias 0 -> 2
- net Net-(D1-K): track 18.0 -> 24.8 mm
- net +5V: track 15.4 -> 9.73 mm
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Other:
- board size 60 x 60 mm -> 76.1 x 60 mm

Commit message: Update
Parts:
- SW1, SW2, SW3: moved to B.Cu
- turned SW1 to 180 degrees
- turned SW2 to 180 degrees
- turned SW3 to 180 degrees
Routing:
- net Net-(U3-IO22): track 44.7 -> 43.8 mm
